Commit message: body builded

File: description/kitti_urdf.xacro (robot description, xacro)
@@ -1,10 +1,88 @@
 <?xml version="1.0"?>
 <robot xmlns:xacro="http://www.ros.org/wiki/xacro"  name="robot">
+  <!-- Specify some colours -->
+  <material name="white">
+    <color rgba="1 1 1 1"/>
+  </material>
+  <material name="red">
+    <color rgba="1 0 0 1"/>
+  </material>
+  <material name="black">
+    <color rgba="0 0 0 1"/>
+  </material>
+  <!-- This link is help to identify the vehicle -->
+  <link name="map">
+    <visual>
+      <origin rpy="0 0 0" xyz="0 0 0"/>
+      <geometry>
+        <sphere radius="0.1"/>
+      </geometry>
+      <material name="red"/>
+    </visual>
+  </link>
   <link name="base_link">
+    <!-- body base -->
     <visual>
+      <origin rpy="0 0 0" xyz="1.355 0 0.4"/>
       <geometry>
-        <cylinder length="0.6" radius="0.2"/>
+        <box size="2.71 1.60 0.8"/>
       </geometry>
     </visual>
+    <!-- body top -->
+    <visual>
+      <origin rpy="0 0 0" xyz="1.355 0 1.1"/>
+      <geometry>
+        <box size="1.355 1.60 0.6"/>
+      </geometry>
+    </visual>
+    <collision>
+      <geometry>
+        <box size="2.71 1.60 1.90"/>
+      </geometry>
+      <origin rpy="0 0 0" xyz="1.355 0 0.65"/>
+    </collision>
+    <!-- front left wheel
+    <visual>
+      <origin rpy="1.570796327 0 0" xyz="2.71 0.8 0"/>
+      <geometry>
+        <cylinder radius="0.3" length="0.225"/>
+      </geometry>
+      <material name="black"/>
+    </visual>
+    -->
+    <!-- front right wheel
+    <visual>
+      <origin rpy="1.570796327 0 0" xyz="2.71 -0.8 0"/>
+      <geometry>
+        <cylinder radius="0.3" length="0.225"/>
+      </geometry>
+      <material name="black"/>
+    </visual>
+    -->
+    <!-- rear left wheel
+    <visual>
+      <origin rpy="1.570796327 0 0" xyz="0 0.8 0"/>
+      <geometry>
+        <cylinder radius="0.3" length="0.225"/>
+      </geometry>
+      <material name="black"/>
+    </visual>
+    -->
+    <!-- rear right wheel
+    <visual>
+      <material name="black"/>
+      <origin rpy="1.570796327 0 0" xyz="0 -0.8 0"/>
+      <geometry>
+        <cylinder radius="0.3" length="0.225"/>
+      </geometry>
+    </visual>
+    -->
   </link>
+  <!-- A simple fixed joint from our empty map link, to our base. -->
+  <!-- The base origin is offset from the map origin -->
+  <joint name="map_to_base_joint" type="fixed">
+    <origin rpy="0 0 0" xyz="0 0 0.3"/>
+    <parent link="map"/>
+    <child link="base_link"/>
+  </joint>
 </robot>

Commit message: Four wheels finished

File: description/kitti_urdf.xacro (robot description, xacro)
@@ -28,4 +28,5 @@
         <box size="2.71 1.60 0.8"/>
       </geometry>
+      <material name="white"/>
     </visual>
     <!-- body top -->
@@ -42,5 +43,5 @@
       <origin rpy="0 0 0" xyz="1.355 0 0.65"/>
     </collision>
-    <!-- front left wheel
+    <!-- front left wheel -->
     <visual>
       <origin rpy="1.570796327 0 0" xyz="2.71 0.8 0"/>
@@ -50,6 +51,5 @@
       <material name="black"/>
     </visual>
-    -->
-    <!-- front right wheel
+    <!-- front right wheel -->
     <visual>
       <origin rpy="1.570796327 0 0" xyz="2.71 -0.8 0"/>
@@ -59,6 +59,5 @@
       <material name="black"/>
     </visual>
-    -->
-    <!-- rear left wheel
+    <!-- rear left wheel -->
     <visual>
       <origin rpy="1.570796327 0 0" xyz="0 0.8 0"/>
@@ -68,6 +67,5 @@
       <material name="black"/>
     </visual>
-    -->
-    <!-- rear right wheel
+    <!-- rear right wheel -->
     <visual>
       <material name="black"/>
@@ -77,5 +75,4 @@
       </geometry>
     </visual>
-    -->
   </link>
   <!-- A simple fixed joint from our empty map link, to our base. -->

Commit message: Develop (#1)
* body builded

* Four wheels finished

* Final version

* update launch

File: description/kitti_urdf.xacro (robot description, xacro)
@@ -1,10 +1,89 @@
 <?xml version="1.0"?>
 <robot xmlns:xacro="http://www.ros.org/wiki/xacro"  name="robot">
+  <!-- Specify some colours -->
+  <material name="white">
+    <color rgba="1 1 1 1"/>
+  </material>
+  <material name="red">
+    <color rgba="1 0 0 1"/>
+  </material>
+  <material name="black">
+    <color rgba="0 0 0 1"/>
+  </material>
+  <!-- This link is help to identify the vehicle -->
+  <!--
+  <link name="map">
+    <visual>
+      <origin rpy="0 0 0" xyz="0 0 0"/>
+      <geometry>
+        <sphere radius="0.1"/>
+      </geometry>
+      <material name="red"/>
+    </visual>
+  </link>
+  -->
   <link name="base_link">
+    <!-- body base -->
     <visual>
+      <origin rpy="0 0 0" xyz="1.355 0 0.4"/>
       <geometry>
-        <cylinder length="0.6" radius="0.2"/>
+        <box size="2.71 1.60 0.8"/>
+      </geometry>
+      <material name="white"/>
+    </visual>
+    <!-- body top -->
+    <visual>
+      <origin rpy="0 0 0" xyz="1.355 0 1.1"/>
+      <geometry>
+        <box size="1.355 1.60 0.6"/>
+      </geometry>
+    </visual>
+    <collision>
+      <geometry>
+        <box size="2.71 1.60 1.90"/>
+      </geometry>
+      <origin rpy="0 0 0" xyz="1.355 0 0.65"/>
+    </collision>
+    <!-- front left wheel -->
+    <visual>
+      <origin rpy="1.570796327 0 0" xyz="2.71 0.8 0"/>
+      <geometry>
+        <cylinder radius="0.3" length="0.225"/>
+      </geometry>
+      <material name="black"/>
+    </visual>
+    <!-- front right wheel -->
+    <visual>
+      <origin rpy="1.570796327 0 0" xyz="2.71 -0.8 0"/>
+      <geometry>
+        <cylinder radius="0.3" length="0.225"/>
+      </geometry>
+      <material name="black"/>
+    </visual>
+    <!-- rear left wheel -->
+    <visual>
+      <origin rpy="1.570796327 0 0" xyz="0 0.8 0"/>
+      <geometry>
+        <cylinder radius="0.3" length="0.225"/>
+      </geometry>
+      <material name="black"/>
+    </visual>
+    <!-- rear right wheel -->
+    <visual>
+      <material name="black"/>
+      <origin rpy="1.570796327 0 0" xyz="0 -0.8 0"/>
+      <geometry>
+        <cylinder radius="0.3" length="0.225"/>
       </geometry>
     </visual>
   </link>
+  <!-- A simple fixed joint from our empty map link, to our base. -->
+  <!-- The base origin is offset from the map origin -->
+  <!--
+  <joint name="map_to_base_joint" type="fixed">
+    <origin rpy="0 0 0" xyz="0 0 0.3"/>
+    <parent link="map"/>
+    <child link="base_link"/>
+  </joint>
+  -->
 </robot>

Commit message: Add camera and lidar

File: description/kitti_urdf.xacro (robot description, xacro)
@@ -3,11 +3,17 @@
   <!-- Specify some colours -->
   <material name="white">
-    <color rgba="1 1 1 1"/>
+    <color rgba="1 1 1 0.8"/>
   </material>
   <material name="red">
-    <color rgba="1 0 0 1"/>
+    <color rgba="1 0 0 0.8"/>
+  </material>
+  <material name="blue">
+    <color rgba="0 0 1 0.8"/>
+  </material>
+  <material name="green">
+    <color rgba="0 1 0 0.8"/>
   </material>
   <material name="black">
-    <color rgba="0 0 0 1"/>
+    <color rgba="0 0 0 0.8"/>
   </material>
   <!-- This link is help to identify the vehicle -->
@@ -87,3 +93,55 @@
   </joint>
   -->
+  <!-- GPS object -->
+  <link name="gps_link">
+    <visual>
+      <geometry>
+        <box size="0.2 0.05 0.05"/>
+      </geometry>
+      <material name="red"/>
+    </visual>
+  </link>
+  <joint name="base_to_gps_joint" type="fixed">
+    <origin rpy="0 0 0" xyz="-0.05 0.32 0.6"/>
+    <parent link="base_link"/>
+    <child link="gps_link"/>
+  </joint>
+  <!-- IMU object -->
+  <link name="imu_link">
+    <!-- Same object with GPS. Only put the link. -->
+  </link>
+  <joint name="base_to_imu_joint" type="fixed">
+    <origin rpy="0 0 0" xyz="-0.05 0.32 0.6"/>
+    <parent link="base_link"/>
+    <child link="imu_link"/>
+  </joint>
+  <!-- LiDAR -->
+  <link name="lidar_link">
+    <visual>
+      <geometry>
+        <cylinder radius="0.1" length="0.15"/>
+      </geometry>
+      <material name="blue"/>
+    </visual>
+  </link>
+  <joint name="imu_to_lidar_joint" type="fixed">
+    <origin rpy="0 0 0" xyz="0.81 -0.32 1.8"/>
+    <parent link="imu_link"/>
+    <child link="lidar_link"/>
+  </joint>
+  <!-- Camera -->
+  <!-- Camera gray left -->
+  <link name="gray_left_camera_link">
+    <visual>
+      <geometry>
+        <box size="0.1 0.05 0.05"/>
+      </geometry>
+      <material name="green"/>
+    </visual>
+  </link>
+  <joint name="lidar_to_gray_left_camera_joint" type="fixed">
+    <origin rpy="0 0 0" xyz="0.27 0 -0.08"/>
+    <parent link="lidar_link"/>
+    <child link="gray_left_camera_link"/>
+  </joint>
 </robot>

Commit message: Add camera link

File: description/kitti_urdf.xacro (robot description, xacro)
@@ -32,11 +32,11 @@
     <!-- body base -->
     <visual>
-      <origin rpy="0 0 0" xyz="1.355 0 0.4"/>
+      <origin rpy="0 0 0" xyz="1.355 0 0.675"/>
       <geometry>
-        <box size="2.71 1.60 0.8"/>
+        <box size="2.71 1.60 1.35"/>
       </geometry>
       <material name="white"/>
     </visual>
-    <!-- body top -->
+    <!-- body top
     <visual>
       <origin rpy="0 0 0" xyz="1.355 0 1.1"/>
@@ -45,9 +45,10 @@
       </geometry>
     </visual>
+    -->
     <collision>
       <geometry>
         <box size="2.71 1.60 1.90"/>
       </geometry>
-      <origin rpy="0 0 0" xyz="1.355 0 0.65"/>
+      <origin rpy="0 0 0" xyz="1.355 0 0.675"/>
     </collision>
     <!-- front left wheel -->
@@ -103,5 +104,5 @@
   </link>
   <joint name="base_to_gps_joint" type="fixed">
-    <origin rpy="0 0 0" xyz="-0.05 0.32 0.6"/>
+    <origin rpy="0 0 0" xyz="-0.05 0.32 0.63"/>
     <parent link="base_link"/>
     <child link="gps_link"/>
@@ -112,5 +113,5 @@
   </link>
   <joint name="base_to_imu_joint" type="fixed">
-    <origin rpy="0 0 0" xyz="-0.05 0.32 0.6"/>
+    <origin rpy="0 0 0" xyz="-0.05 0.32 0.63"/>
     <parent link="base_link"/>
     <child link="imu_link"/>
@@ -126,5 +127,5 @@
   </link>
   <joint name="imu_to_lidar_joint" type="fixed">
-    <origin rpy="0 0 0" xyz="0.81 -0.32 1.8"/>
+    <origin rpy="0 0 0" xyz="0.81 -0.32 0.8"/>  <!-- okay! double checked. -->
     <parent link="imu_link"/>
     <child link="lidar_link"/>
@@ -134,4 +135,21 @@
   <link name="gray_left_camera_link">
     <visual>
+      <origin rpy="0 0 0" xyz="0 0 0"/>
+      <geometry>
+        <box size="0.05 0.05 0.1"/>
+      </geometry>
+      <material name="green"/>
+    </visual>
+  </link>
+  <joint name="lidar_to_gray_left_camera_joint" type="fixed">
+    <!-- warning!!! the coordinate is different!!! -->
+    <!-- x: pointing right, y: pointing down, z: pointint front-->
+    <origin rpy="-1.570796327 0 -1.570796327" xyz="0.27 0 -0.08"/>
+    <parent link="lidar_link"/>
+    <child link="gray_left_camera_link"/>
+  </joint>
+  <!-- Camera color left
+  <link name="color_left_camera_link">
+    <visual>
       <geometry>
         <box size="0.1 0.05 0.05"/>
@@ -140,8 +158,9 @@
     </visual>
   </link>
-  <joint name="lidar_to_gray_left_camera_joint" type="fixed">
-    <origin rpy="0 0 0" xyz="0.27 0 -0.08"/>
-    <parent link="lidar_link"/>
-    <child link="gray_left_camera_link"/>
+  <joint name="gray_left_camera_to_color_left_joint" type="fixed">
+    <origin rpy="0 0 0" xyz="0 0.06 0"/>
+    <parent link="gray_left_camera_link"/>
+    <child link="color_left_camera_link"/>
   </joint>
+  -->
 </robot>

Commit message: Add all cameras

File: description/kitti_urdf.xacro (robot description, xacro)
@@ -17,20 +17,9 @@
     <color rgba="0 0 0 0.8"/>
   </material>
-  <!-- This link is help to identify the vehicle -->
-  <!--
-  <link name="map">
-    <visual>
-      <origin rpy="0 0 0" xyz="0 0 0"/>
-      <geometry>
-        <sphere radius="0.1"/>
-      </geometry>
-      <material name="red"/>
-    </visual>
-  </link>
-  -->
+  <!-- body of the vehicle -->
   <link name="base_link">
     <!-- body base -->
     <visual>
-      <origin rpy="0 0 0" xyz="1.355 0 0.675"/>
+      <origin xyz="1.355 0 0.675"/>
       <geometry>
         <box size="2.71 1.60 1.35"/>
@@ -48,7 +37,7 @@
     <collision>
       <geometry>
+      <origin xyz="1.355 0 0.675"/>
         <box size="2.71 1.60 1.90"/>
       </geometry>
-      <origin rpy="0 0 0" xyz="1.355 0 0.675"/>
     </collision>
     <!-- front left wheel -->
@@ -85,13 +74,4 @@
     </visual>
   </link>
-  <!-- A simple fixed joint from our empty map link, to our base. -->
-  <!-- The base origin is offset from the map origin -->
-  <!--
-  <joint name="map_to_base_joint" type="fixed">
-    <origin rpy="0 0 0" xyz="0 0 0.3"/>
-    <parent link="map"/>
-    <child link="base_link"/>
-  </joint>
-  -->
   <!-- GPS object -->
   <link name="gps_link">
@@ -104,5 +84,5 @@
   </link>
   <joint name="base_to_gps_joint" type="fixed">
-    <origin rpy="0 0 0" xyz="-0.05 0.32 0.63"/>
+    <origin xyz="-0.05 0.32 0.63"/>
     <parent link="base_link"/>
     <child link="gps_link"/>
@@ -113,5 +93,5 @@
   </link>
   <joint name="base_to_imu_joint" type="fixed">
-    <origin rpy="0 0 0" xyz="-0.05 0.32 0.63"/>
+    <origin xyz="-0.05 0.32 0.63"/>
     <parent link="base_link"/>
     <child link="imu_link"/>
@@ -127,13 +107,12 @@
   </link>
   <joint name="imu_to_lidar_joint" type="fixed">
-    <origin rpy="0 0 0" xyz="0.81 -0.32 0.8"/>  <!-- okay! double checked. -->
+    <origin xyz="0.81 -0.32 0.8"/>  <!-- okay! double checked. -->
     <parent link="imu_link"/>
     <child link="lidar_link"/>
   </joint>
   <!-- Camera -->
-  <!-- Camera gray left -->
-  <link name="gray_left_camera_link">
+  <!-- Camera 0 (gray left) -->
+  <link name="camera0_link">
     <visual>
-      <origin rpy="0 0 0" xyz="0 0 0"/>
       <geometry>
         <box size="0.05 0.05 0.1"/>
@@ -142,25 +121,51 @@
     </visual>
   </link>
-  <joint name="lidar_to_gray_left_camera_joint" type="fixed">
-    <!-- warning!!! the coordinate is different!!! -->
+  <joint name="lidar_to_camera0_joint" type="fixed">
     <!-- x: pointing right, y: pointing down, z: pointint front-->
     <origin rpy="-1.570796327 0 -1.570796327" xyz="0.27 0 -0.08"/>
     <parent link="lidar_link"/>
-    <child link="gray_left_camera_link"/>
+    <child link="camera0_link"/>
   </joint>
-  <!-- Camera color left
-  <link name="color_left_camera_link">
+  <!-- Camera 1 (gray right) -->
+  <link name="camera1_link">
     <visual>
       <geometry>
-        <box size="0.1 0.05 0.05"/>
+        <box size="0.05 0.05 0.1"/>
       </geometry>
       <material name="green"/>
     </visual>
   </link>
-  <joint name="gray_left_camera_to_color_left_joint" type="fixed">
-    <origin rpy="0 0 0" xyz="0 0.06 0"/>
-    <parent link="gray_left_camera_link"/>
-    <child link="color_left_camera_link"/>
+  <joint name="camera0_to_camera1_joint" type="fixed">
+    <origin xyz="0.54 0 0"/>
+    <parent link="camera0_link"/>
+    <child link="camera1_link"/>
   </joint>
-  -->
+  <!-- Camera 2 (color left) -->
+  <link name="camera2_link">
+    <visual>
+      <geometry>
+        <box size="0.05 0.05 0.1"/>
+      </geometry>
+      <material name="green"/>
+    </visual>
+  </link>
+  <joint name="camera0_to_camera2" type="fixed">
+    <origin xyz="-0.06 0 0"/>
+    <parent link="camera0_link"/>
+    <child link="camera2_link"/>
+  </joint>
+  <!-- Camera 3 (color right) -->
+  <link name="camera3_link">
+    <visual>
+      <geometry>
+        <box size="0.05 0.05 0.1"/>
+      </geometry>
+      <material name="green"/>
+    </visual>
+  </link>
+  <joint name="camera0_to_camera3" type="fixed">
+    <origin xyz="0.48 0 0"/>
+    <parent link="camera0_link"/>
+    <child link="camera3_link"/>
+  </joint>
 </robot>

Commit message: Finished

File: description/kitti_urdf.xacro (robot description, xacro)
@@ -18,10 +18,15 @@
   </material>
   <!-- body of the vehicle -->
+  <xacro:property name="vehicle_length" value="2.71"/>
+  <xacro:property name="vehicle_width" value="1.60"/>
+  <xacro:property name="vehicle_height" value="1.35"/>
+  <xacro:property name="wheel_radius" value="0.3"/>
+  <xacro:property name="wheel_length" value="0.225"/>
   <link name="base_link">
     <!-- body base -->
     <visual>
-      <origin xyz="1.355 0 0.675"/>
+      <origin xyz="${vehicle_length/2} 0 ${vehicle_height/2}"/>
       <geometry>
-        <box size="2.71 1.60 1.35"/>
+        <box size="${vehicle_length} ${vehicle_width} ${vehicle_height}"/>
       </geometry>
       <material name="white"/>
@@ -36,14 +41,15 @@
     -->
     <collision>
+      <origin xyz="${vehicle_length/2} 0 ${vehicle_height/2}"/>
       <geometry>
-      <origin xyz="1.355 0 0.675"/>
-        <box size="2.71 1.60 1.90"/>
+        <box size="${vehicle_length} ${vehicle_width} ${vehicle_height}"/>
       </geometry>
     </collision>
+    <!-- Wheel -->
     <!-- front left wheel -->
     <visual>
-      <origin rpy="1.570796327 0 0" xyz="2.71 0.8 0"/>
+      <origin rpy="${pi/2} 0 0" xyz="${vehicle_length} ${vehicle_width/2} 0"/>
       <geometry>
-        <cylinder radius="0.3" length="0.225"/>
+        <cylinder radius="${wheel_radius}" length="${wheel_length}"/>
       </geometry>
       <material name="black"/>
@@ -51,7 +57,7 @@
     <!-- front right wheel -->
     <visual>
-      <origin rpy="1.570796327 0 0" xyz="2.71 -0.8 0"/>
+      <origin rpy="${pi/2} 0 0" xyz="${vehicle_length} ${-vehicle_width/2} 0"/>
       <geometry>
-        <cylinder radius="0.3" length="0.225"/>
+        <cylinder radius="${wheel_radius}" length="${wheel_length}"/>
       </geometry>
       <material name="black"/>
@@ -59,7 +65,7 @@
     <!-- rear left wheel -->
     <visual>
-      <origin rpy="1.570796327 0 0" xyz="0 0.8 0"/>
+      <origin rpy="${pi/2} 0 0" xyz="0 ${vehicle_width/2} 0"/>
       <geometry>
-        <cylinder radius="0.3" length="0.225"/>
+        <cylinder radius="${wheel_radius}" length="${wheel_length}"/>
       </geometry>
       <material name="black"/>
@@ -68,7 +74,7 @@
     <visual>
       <material name="black"/>
-      <origin rpy="1.570796327 0 0" xyz="0 -0.8 0"/>
+      <origin rpy="${pi/2} 0 0" xyz="0 ${-vehicle_width/2} 0"/>
       <geometry>
-        <cylinder radius="0.3" length="0.225"/>
+        <cylinder radius="${wheel_radius}" length="${wheel_length}"/>
       </geometry>
     </visual>
@@ -107,14 +113,17 @@
   </link>
   <joint name="imu_to_lidar_joint" type="fixed">
-    <origin xyz="0.81 -0.32 0.8"/>  <!-- okay! double checked. -->
+    <origin xyz="0.81 -0.32 0.8"/>
     <parent link="imu_link"/>
     <child link="lidar_link"/>
   </joint>
   <!-- Camera -->
+  <xacro:property name="camera_length" value="0.05"/>
+  <xacro:property name="camera_width" value="0.05"/>
+  <xacro:property name="camera_height" value="0.1"/>
   <!-- Camera 0 (gray left) -->
   <link name="camera0_link">
     <visual>
       <geometry>
-        <box size="0.05 0.05 0.1"/>
+        <box size="${camera_length} ${camera_width} ${camera_height}"/>
       </geometry>
       <material name="green"/>
@@ -123,5 +132,5 @@
   <joint name="lidar_to_camera0_joint" type="fixed">
     <!-- x: pointing right, y: pointing down, z: pointint front-->
-    <origin rpy="-1.570796327 0 -1.570796327" xyz="0.27 0 -0.08"/>
+    <origin rpy="${-pi/2} 0 ${-pi/2}" xyz="0.27 0 -0.08"/>
     <parent link="lidar_link"/>
     <child link="camera0_link"/>
@@ -131,5 +140,5 @@
     <visual>
       <geometry>
-        <box size="0.05 0.05 0.1"/>
+        <box size="${camera_length} ${camera_width} ${camera_height}"/>
       </geometry>
       <material name="green"/>
@@ -145,5 +154,5 @@
     <visual>
       <geometry>
-        <box size="0.05 0.05 0.1"/>
+        <box size="${camera_length} ${camera_width} ${camera_height}"/>
       </geometry>
       <material name="green"/>
@@ -159,5 +168,5 @@
     <visual>
       <geometry>
-        <box size="0.05 0.05 0.1"/>
+        <box size="${camera_length} ${camera_width} ${camera_height}"/>
       </geometry>
       <material name="green"/>
